Commit message: fix: BlackShipに合わせてサイズを変更

File: urdf/blackship_body.urdf (robot description, URDF)
Before this commit: robot BlackShip, 6 links, 5 joints
Links:
- removed link ball_link
- added link lidar_support_link; visual box size=0.05 0.33 0.4
- link body_link: geometry visual box size=0.5 0.33 0.25
- link left_wheeel_link: geometry visual cylinder length=0.04 radius=0.085
- link right_wheeel_link: geometry visual cylinder length=0.04 radius=0.085
Joints:
- removed joint ball_joint
- added joint lidar_support_joint: type fixed, parent body_link, child lidar_support_link, origin xyz=0.15 0 0.325
- joint body_joint: origin xyz=0.075 0 0.05 -> xyz=0.0 0 0.1675
- joint left_wheel_joint: origin xyz=0 0.09 0.025 rpy=-1.57 0 0 -> xyz=0 0.167 -0.125 rpy=-1.57 0 0
- joint lidar_joint: origin xyz=0.125 0 0.1 -> xyz=0.15 0 0.54
- joint right_wheel_joint: origin xyz=0 -0.09 0.025 rpy=-1.57 0 0 -> xyz=0 -0.167 -0.125 rpy=-1.57 0 0
